File: Boards/Central_ECU/ign+nc_valve.kicad_sch (KiCad schematic)
At the start: 31 parts, among them Q1 DMT12H060LFDF, U4 LM339B, U5 LM1084-ADJ, U6 TPS16630PWPR

Commit message: Central ECU to order
Parts:
- removed C21: 10u, Capacitor_SMD:C_0603_1608Metric, symbol Device:C
- removed C22: 50u, Capacitor_SMD:CP_Elec_6.3x9.9, symbol Device:C_Polarized
- removed R24: 1K40, Resistor_SMD:R_0603_1608Metric, symbol Device:R
- removed U5: LM1084-ADJ, Package_TO_SOT_SMD:TO-263-3_TabPin2, symbol Regulator_Linear:LM1084-ADJ
- added C43: 100u, Capacitor_SMD:CP_Elec_8x10.5, symbol Device:C_Polarized
- added D16: 30V 34VC, Diode_SMD:D_SOD-882, symbol Device:D_TVS
- added J16: MICROFIT, Connector_Molex:Molex_Micro-Fit_3.0_43045-0412_2x02_P3.00mm_Vertical, symbol Connector_Generic:Conn_02x02_Counter_Clockwise
- C23, C24: value 22u -> 10u; footprint Capacitor_SMD:C_0603_1608Metric -> Capacitor_SMD:C_1206_3216Metric
- C27: value 22u -> 10u
- R20: now fitted
- R21, R22: now not fitted
- R23: value 121R -> 0R; footprint Resistor_SMD:R_0603_1608Metric -> Resistor_SMD:R_1206_3216Metric
- TP29: value 12V -> SPICY+
Connections:
- net GND: now also C43.2, D16.1 (A1), J16.2 (Pin_2), J16.3 (Pin_3)
- net Pyro Low Side/Ign+: now also R23.2; no longer C27.1, F1.1, R27.2, U6.18 (OUT), U6.19 (OUT), U6.20 (OUT)
- net at R21.2: now also J16.1 (Pin_1)
- net at R23.1: now also C27.1, F1.1, R27.2, U6.18 (OUT), U6.19 (OUT), U6.20 (OUT); no longer R22.1
- new net: C43.1, D16.2 (A2), J16.4 (Pin_4), R22.1
Other:
- note added: "ABS MAX 36V DIODE MAX 30V"
- note added: "Bypassed battery voltage or connector for external regualtor"
- note added: "External Regulator"
- note added: "Resistor for possible current limiting. May be issue with high voltage where ignitor leads melt before end."
- note added: "To allow for 8s battery connection (33.6V max) change TVS to PESD1CANFD33L-QYL"
- note removed: "12V Regulator"
- note removed: "Bypass to allow for externally regulated power to be passed directly through. This will be useful if a 24V solenoid is used."
- note removed: "Efficiency with 4s lipo input: Worst case 12/16.8 = 71% Typical case 12/14.8 = 81% Max power loss (16w servo) = 6.6W"
- note removed: "Output requires some ESR for stablilty, namely zero at 50kHz. Datasheet reccomends 10u tantalum or 50u electrolytic. Could also look at ceramic with series resistor as per https://www.ti.com/document-viewer/lit/html/SSZTBJ1"
- note removed: "Vout = 1.25(1+R2/R1)"
- moved on the sheet: TP30
