File: Boards/Central_ECU/Central_ECU.kicad_pcb (KiCad board)
At the start: 4 copper layers, 100 x 100 mm, 180 parts, among them J1 Micro_SD_Card, J10 Solenoid NANOFIT, J11 DB9 Microfit, J12 RS422 JST, J13 USB_B_Micro, J14 SWD JST PH, J15 UART JST, J16 MICROFIT, J2 Extras JST, J3 MICROFIT, J4 Siren MICROFIT, J5 I2CB JST, J6 MICROFIT, J7 I2CA JST, J8 Ignitor JST EH, J9 DB9 MICROFIT, Q1 DMT12H060LFDF, Q2 DMT12H060LFDF, Q3 DMT12H060LFDF, Q4 DMP6023LFG, Q5 DMP6023LFG, SW1 Arm Switch, SW2 On Switch, U1 SSD1306, U2 STM32G0B1RCTx, U3 TCAN1046, U4 LM339B, U6 TPS16630PWPR, U7 AZ1117C-5.0, U8 AZ1117C-3.3, U9 LPS22HH, Y1 8MHz, Y2 32.768k

Commit message: Updated resistors on ECU, added code to read battery voltages
Parts:
- R10, R12, R8, R9: value 60R -> 60.4R
- R44: value 10K2 -> 18K
- R45: value 2K49 -> 2K7
- TP2: value ADC4S -> ADC6S
Connections:
- net /ADC_0 (4S) renamed /ADC_0 (6S)
Changed lines of the file:
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@@
 	(net 93 "/OX_LOW_SENSE")
 	(net 94 "/EMATCH_1_CONT")
-	(net 95 "/ADC_0 (4S)")
+	(net 95 "/ADC_0 (6S)")
 	(net 96 "/ADC_1 (2S)")
 	(net 97 "/CAN1_RX")
@@
 			)
 		)
-		(property "Value" "10K2"
+		(property "Value" "18K"
 			(at 0 1.43 0)
 			(layer "F.Fab")
@@
 			(layers "F.Cu" "F.Mask" "F.Paste")
 			(roundrect_rratio 0.25)
-			(net 95 "/ADC_0 (4S)")
+			(net 95 "/ADC_0 (6S)")
 			(pintype "passive")
 		)
@@
 			)
 		)
-		(property "Value" "60R"
+		(property "Value" "60.4R"
 			(at 0 1.43 0)
 			(layer "F.Fab")
@@
 			)
 		)
-		(property "Value" "2K49"
+		(property "Value" "2K7"
 			(at 0 1.43 0)
 			(layer "F.Fab")
@@
 			(layers "F.Cu" "F.Mask" "F.Paste")
 			(roundrect_rratio 0.25)
-			(net 95 "/ADC_0 (4S)")
+			(net 95 "/ADC_0 (6S)")
 			(pintype "passive")
 		)
@@
 			)
 		)
-		(property "Value" "60R"
+		(property "Value" "60.4R"
 			(at 0 1.43 0)
 			(layer "F.Fab")
@@
 			)
 		)
-		(property "MPN" "B4B-PH-K-S"
+		(property "MPN" "B4B-EH-A"
 			(at 0 0 0)
 			(unlocked yes)
@@
 			)
 		)
-		(property "Value" "ADC4S"
+		(property "Value" "ADC6S"
 			(at 0 1.75 0)
 			(layer "F.SilkS")
@@
 			(size 1.5 1.5)
 			(layers "F.Cu" "F.Mask")
-			(net 95 "/ADC_0 (4S)")
+			(net 95 "/ADC_0 (6S)")
 			(pinfunction "1")
 			(pintype "passive")
@@
 			(layers "F.Cu" "F.Mask" "F.Paste")
 			(roundrect_rratio 0.25)
-			(net 95 "/ADC_0 (4S)")
+			(net 95 "/ADC_0 (6S)")
 			(pinfunction "PA0")
 			(pintype "bidirectional")
@@
 			)
 		)
-		(property "Value" "60R"
+		(property "Value" "60.4R"
 			(at 0 1.43 0)
 			(layer "F.Fab")
@@
 			)
 		)
-		(property "Value" "60R"
+		(property "Value" "60.4R"
 			(at 0 1.43 0)
 			(layer "F.Fab")

Commit message: Changes to reflect incorrect schematic labeling
Connections:
- CR1 pad 5: /422D_N -> /422D_P
- CR1 pad 6: /422D_P -> /422D_N
- J12 pad 4: /422D_P -> /422D_N
- J12 pad 5: /422D_N -> /422D_P
- TP10 pad 1: /CAN2_RX -> /CAN1_RX
- TP11 pad 1: /CAN2_TX -> /CAN1_RX
- TP8 pad 1: /CAN1_TX -> /CAN1_RX
- U2 pad 25: /CAN2_RX -> /CAN1_RX
- U2 pad 26: /CAN2_TX -> /CAN1_RX
- U2 pad 27: /CAN1_RX -> /CAN2_RX
- U2 pad 28: /CAN1_TX -> /CAN2_TX
- U3 pad 4: /CAN1_TX -> /CAN1_RX
- U3 pad 6: /CAN2_RX -> /CAN1_RX
- U3 pad 7: /CAN2_TX -> /CAN1_RX
Routing:
- net /CAN1_RX: track 22.8 -> 72.8 mm
- net /CAN2_RX: track 26.5 -> 0.00 mm
- net /CAN1_TX: track 26.3 -> 0.00 mm
- net (no net): track 0.00 -> 26.3 mm
- net /CAN2_TX: track 23.6 -> 0.00 mm
