File: Boards/Servo_Board/Servo_Board.kicad_sch (KiCad schematic)
At the start: 44 parts, among them J1 DE9_Pins, J10 Conn_01x04, J11 Conn_01x04, J12 Conn_01x04, J13 Conn_01x04, J14 Conn_01x04, J15 Conn_01x04, J16 Conn_01x04, J2 USB_B_Micro, J3 Conn_02x05_Odd_Even, J9 DE9_Socket, U1 STM32G0B1RCTx, U5 BD50HC5WEFJ-E2, Y2 Crystal 8MHz

Commit message: Ongoing changes to satellite  boards and test code
Parts:
- removed C15, C16: 1u, Capacitor_SMD:C_0603_1608Metric, symbol Device:C
- removed C17: 4.7u, Capacitor_SMD:C_0603_1608Metric, symbol Device:C
- removed C18: 100n, Capacitor_SMD:C_0603_1608Metric, symbol Device:C
- removed D1, D2, D3, D4, D5, D6, D7: D_Schottky, Diode_SMD:D_SOD-882, symbol Device:D_Schottky
- removed J1: DE9_Pins, Connector_Molex:Molex_Micro-Fit_3.0_43650-0915_1x09_P3.00mm_Vertical, symbol Connector:DE9_Pins
- removed J10, J11, J12, J13, J14, J15, J16: Conn_01x04, Connector_Molex:Molex_Micro-Fit_3.0_43045-0412_2x02_P3.00mm_Vertical, symbol Connector_Generic:Conn_01x04
- removed J2: USB_B_Micro, Connector_USB:USB_Micro-AB_Molex_47590-0001, symbol Connector:USB_B_Micro
- removed J3: Conn_02x05_Odd_Even, Connector_IDC:IDC-Header_2x05_P2.54mm_Vertical, symbol Connector_Generic:Conn_02x05_Odd_Even
- removed J9: DE9_Socket, Connector_Molex:Molex_Micro-Fit_3.0_43650-0915_1x09_P3.00mm_Vertical, symbol Connector:DE9_Socket
- removed JP1, JP2: Jumper_2_Bridged, Connector_PinSocket_2.54mm:PinSocket_1x02_P2.54mm_Vertical, symbol Jumper:Jumper_2_Bridged
- removed U1: STM32G0B1RCTx, Package_QFP:LQFP-64_10x10mm_P0.5mm, symbol MCU_ST_STM32G0:STM32G0B1RCTx
- removed U3: ~, footprints:TSOT23-5_ONS, symbol 0_Custom_Symbols:CAT6219
- removed U4: ~, footprints:SOT23_DYY_TEX, symbol Interface_CAN_LIN:TCAN1046AV-Q1
- removed U5: BD50HC5WEFJ-E2, footprints:HTSOP-J8_ROM, symbol 0_Custom_Symbols:BD50HC5WEFJ-E2
- removed Y2: Crystal 8MHz, Crystal:Crystal_SMD_Abracon_ABM3B-4Pin_5.0x3.2mm, symbol Device:Crystal
- added C1: 100u, Capacitor_SMD:CP_Elec_8x10.5, symbol Device:C_Polarized
- added C2, C4: 10u, Capacitor_SMD:C_0603_1608Metric, symbol Device:C
- added C3, C5: 22u, Capacitor_SMD:C_1206_3216Metric, symbol Device:C
- added D1: 9V 15.4VC, Diode_SMD:D_SOD-123F, symbol Device:D_TVS
- added D2: 18V, Diode_SMD:D_SOD-323F, symbol Device:D_Zener
- added D3, D4: PESD3V3L4UW, Package_TO_SOT_SMD:SOT-665, symbol Power_Protection:PESD3V3L4UW
- added F1, F2: 2A, symbol Device:Fuse
- added H1, H2, H3, H4: ~, MountingHole:MountingHole_3.2mm_M3_DIN965_Pad_TopOnly, symbol Mechanical:MountingHole_Pad
- added J1, J2: DB9 Microfit, Connector_Molex:Molex_Micro-Fit_3.0_43045-1012_2x05_P3.00mm_Vertical, symbol Connector:DE9_Socket
- added J10: I2CA JST, Connector_JST:JST_PH_B5B-PH-K_1x05_P2.00mm_Vertical, symbol Connector_Generic:Conn_01x05
- added J11: I2CB JST, Connector_JST:JST_PH_B5B-PH-K_1x05_P2.00mm_Vertical, symbol Connector_Generic:Conn_01x05
- added J12: I2CC JST, Connector_JST:JST_PH_B5B-PH-K_1x05_P2.00mm_Vertical, symbol Connector_Generic:Conn_01x05
- added J13: SERVO A, Connector_Molex:Molex_Micro-Fit_3.0_43045-0412_2x02_P3.00mm_Vertical, symbol Connector_Generic:Conn_02x02_Counter_Clockwise
- added J14: SERVO B, Connector_Molex:Molex_Micro-Fit_3.0_43045-0412_2x02_P3.00mm_Vertical, symbol Connector_Generic:Conn_02x02_Counter_Clockwise
- added J15: SERVO C, Connector_Molex:Molex_Micro-Fit_3.0_43045-0412_2x02_P3.00mm_Vertical, symbol Connector_Generic:Conn_02x02_Counter_Clockwise
- added J16: SERVO D, Connector_Molex:Molex_Micro-Fit_3.0_43045-0412_2x02_P3.00mm_Vertical, symbol Connector_Generic:Conn_02x02_Counter_Clockwise
- added J3, J4: CAN1_T, Connector_PinHeader_2.54mm:PinHeader_1x02_P2.54mm_Vertical, symbol Connector_Generic:Conn_01x02
- added J5: USB_B_Micro, Connector_USB:USB_Micro-B_Amphenol_10118193-0001LF_Horizontal, symbol Connector:USB_B_Micro
- added J6: SWD JST PH, Connector_JST:JST_PH_B4B-PH-K_1x04_P2.00mm_Vertical, symbol Connector_Generic:Conn_01x04
- added J7: UART JST, Connector_JST:JST_PH_B3B-PH-K_1x03_P2.00mm_Vertical, symbol Connector_Generic:Conn_01x03
- added J8: AUX BATT CONN, Connector_JST:JST_PH_B4B-PH-K_1x04_P2.00mm_Vertical, symbol Connector_Generic:Conn_01x04
- added J9: Extras JST, Connector_JST:JST_PH_B7B-PH-K_1x07_P2.00mm_Vertical, symbol Connector_Generic:Conn_01x07
- added JP1: CH SEL, symbol Jumper:SolderJumper_3_Bridged12
- added JP2: CL SEL, symbol Jumper:SolderJumper_3_Bridged12
- added Q1: DMP6023LFG, Package_SON:Diodes_PowerDI3333-8, symbol Transistor_FET:DMP3013SFV
- added R10: 14K3, Resistor_SMD:R_0603_1608Metric, symbol Device:R
- added R11: 9K53, Resistor_SMD:R_0603_1608Metric, symbol Device:R
- added R12, R13, R14: 0R, Resistor_SMD:R_0603_1608Metric, symbol Device:R
- added R7: 27R, Resistor_SMD:R_0603_1608Metric, symbol Device:R
- added R8: 120R, symbol Device:R
- added R9: 100K, Resistor_SMD:R_0603_1608Metric, symbol Device:R
- added TP14: RS422TX, TestPoint:TestPoint_Pad_1.5x1.5mm, symbol Connector:TestPoint_Small
- added TP16: RS422RX, TestPoint:TestPoint_Pad_1.5x1.5mm, symbol Connector:TestPoint_Small
- added TP2: ADC4S, TestPoint:TestPoint_Pad_1.5x1.5mm, symbol Connector:TestPoint_Small
- added TP3: ADC2S, TestPoint:TestPoint_Pad_1.5x1.5mm, symbol Connector:TestPoint_Small
- added TP31: ADC2, TestPoint:TestPoint_Pad_1.5x1.5mm, symbol Connector:TestPoint_Small
- added TP32: ADC3, TestPoint:TestPoint_Pad_1.5x1.5mm, symbol Connector:TestPoint_Small
- added TP4: SPISCK, TestPoint:TestPoint_Pad_1.5x1.5mm, symbol Connector:TestPoint_Small
- added TP5: SPIMISO, TestPoint:TestPoint_Pad_1.5x1.5mm, symbol Connector:TestPoint_Small
- added TP7: SPICS, TestPoint:TestPoint_Pad_1.5x1.5mm, symbol Connector:TestPoint_Small
- added TP8: CANTX1, TestPoint:TestPoint_Pad_1.5x1.5mm, symbol Connector:TestPoint_Small
- added TP9: CANRX1, TestPoint:TestPoint_Pad_1.5x1.5mm, symbol Connector:TestPoint_Small
- added U1: AZ1117C-5.0, Package_TO_SOT_SMD:SOT-223-3_TabPin2, symbol Regulator_Linear:AZ1117-5.0
- added U2: STM32G0B1RCTx, Package_QFP:LQFP-64_10x10mm_P0.5mm, symbol MCU_ST_STM32G0:STM32G0B1RCTx
- added U3: TCAN1046, Custom:SOT23_DYY_TEX, symbol Interface_CAN_LIN:TCAN1046AV-Q1
- added U4: AZ1117C-3.3, Package_TO_SOT_SMD:SOT-223-3_TabPin2, symbol Regulator_Linear:AZ1117-3.3
- added Y1: 8MHz, Crystal:Crystal_SMD_Abracon_ABM8G-4Pin_3.2x2.5mm, symbol Device:Crystal
- C10: value 100n -> 4u7
- C11, C12: value 100n -> ?; footprint Capacitor_SMD:C_0603_1608Metric -> Capacitor_SMD:C_0402_1005Metric; now not fitted; now left out of the parts list
- C13: value 4u7 -> 100n
- C6: value 10u -> 100n; footprint Capacitor_SMD:C_0603_1608Metric -> Capacitor_SMD:C_0402_1005Metric
- C7: value 10u -> 4u7
- C8, C9: value 20p -> 100n; footprint Capacitor_SMD:C_0603_1608Metric -> Capacitor_SMD:C_0402_1005Metric
- R1, R2, R3, R4: value 60 -> 100K; footprint Resistor_SMD:R_0603_1608Metric -> (none)
- R5: value 27R -> 120R; footprint Resistor_SMD:R_0603_1608Metric -> (none)
Connections:
- net D_N is gone; now on net CANH2: R5.2
- net CAN1_RX: now also TP9.1, U2.27 (PB0), U3.1 (TXD1)
- net CAN1_TX: now also TP8.1, U2.28 (PB1), U3.4 (RXD1)
- net CANH1: now also J1.6, J2.6, J3.1 (Pin_1), JP1.1 (A); no longer R1.1
- net CANH2: now also J1.8, J2.8, JP1.3 (B); no longer R3.1
- net CANL1: now also J1.7, J2.7, J4.1 (Pin_1), JP2.1 (A); no longer R2.2
- net CANL2: now also J1.9, J2.9, JP2.3 (B), R8.2; no longer R4.2
- net GND: now also C1.2, C2.2, C3.2, C4.2, C5.2, D1.1 (A1), D3.2 (A), D4.2 (A), H1.1, H2.1, H3.1, H4.1, J1.2, J1.4, J10.1 (Pin_1), J11.1 (Pin_1), J12.1 (Pin_1), J13.3 (Pin_3), J14.3 (Pin_3), J15.3 (Pin_3), J16.3 (Pin_3), J2.2, J2.4, J5.5 (GND), J6.2 (Pin_2), J7.2 (Pin_2), J8.3 (Pin_3), J8.4 (Pin_4), J9.1 (Pin_1), J9.7 (Pin_7), R11.2, R9.2, U1.1 (GND), U2.9 (VSS), U3.2 (GND), U3.5 (GND), U4.1 (GND)
- net SWCLK: now also J6.1 (Pin_1), U2.46 (PA14)
- net SWDIO: now also J6.3 (Pin_3), U2.45 (PA13)
- net +3V3: now reaches C9.1
- net +3V3: now also C10.1, C14.1, C6.1, C7.1, C8.1, R1.1, R2.1, R3.2, R4.2, C5.1, J10.5 (Pin_5), J11.5 (Pin_5), J12.5 (Pin_5), R12.1, U2.6 (VBAT), U2.7 (VREF+), U2.8 (VDD), U3.11 (VIO), U4.2 (VO)
- net at R1.2: now also U3.6 (TXD2)
- net at R5.1: now also J3.2 (Pin_2)
- net at R4.1: now also U3.14 (STB1)
- net at R6.1: now also U2.43 (PA9/PA11)
- removed net 3V3: C10.1, C12.1, C13.1, C14.1, C7.1
- net 5V: no longer names the net of C11.1
- net 5V: now also U2.10 (PF0), Y1.1; no longer C6.1
- net D_P renamed USB_D-
- net USB_D-: now also J5.2 (D-)
- new net: C12.1, U2.11 (PF1), Y1.3 (2)
- new net: D2.2 (A), Q1.4 (G), R9.1
- new net: D1.2 (A2), F1.1, F2.2, Q1.5 (D)
- new net: J9.4 (Pin_4), R12.2, R13.2, R14.2
- new net: R2.2, U3.7 (RXD2)
- new net: R3.1, U3.8 (STB2)
- new net: F2.1, J8.1 (Pin_1), J8.2 (Pin_2)
- new net: R7.1, U2.44 (PA10/PA12)
- new net: J4.2 (Pin_2), R8.1
- new net +5V: C13.1, C3.1, C4.1, J10.3 (Pin_3), J11.3 (Pin_3), J12.3 (Pin_3), R13.1, U1.2 (VO), U3.3 (VCC), U4.3 (VI)
- new net +7V4: C1.1, C2.1, D2.1 (K), J13.1 (Pin_1), J14.1 (Pin_1), J15.1 (Pin_1), J16.1 (Pin_1), Q1.1 (S), Q1.2 (S), Q1.3 (S), R10.1, R14.1, U1.3 (VI)
- new net +7V4_CAN: F1.2, J1.1, J1.5, J2.1, J2.5
- new net 2S_VOLTAGE: R10.2, R11.1
- new net ADC_0 (4S): TP2.1, U2.17 (PA0)
- new net ADC_1 (2S): TP3.1, U2.18 (PA1)
- new net ADC_2: TP31.1, U2.19 (PA2)
- new net ADC_3: TP32.1, U2.20 (PA3)
- new net CAN1_AUX: J1.3, U2.33 (PB13)
- new net CAN2_AUX: J2.3, U2.32 (PB12)
- new net CANH: JP1.2 (C), U3.13 (CANH1)
- new net CANL: JP2.2 (C), U3.12 (CANL1)
- new net E1: J9.2 (Pin_2), U2.51 (PD1)
- new net E2: J9.3 (Pin_3), U2.52 (PD2)
- new net E3: J9.5 (Pin_5), U2.53 (PD3)
- new net E4: J9.6 (Pin_6), U2.54 (PD4)
- new net I2C1_SCL: D3.3 (K2), J10.4 (Pin_4), U2.62 (PB8)
- new net I2C1_SDA: D3.1 (K1), J10.2 (Pin_2), U2.63 (PB9)
- new net I2C2_SCL: D3.5 (K4), J11.4 (Pin_4), U2.57 (PB3)
- new net I2C2_SDA: D3.4 (K3), J11.2 (Pin_2), U2.58 (PB4)
- new net I2C3_SCL: D4.3 (K2), J12.4 (Pin_4), U2.13 (PC0)
- new net I2C3_SDA: D4.1 (K1), J12.2 (Pin_2), U2.14 (PC1)
- new net LED1: U2.50 (PD0)
- new net NRST: J6.4 (Pin_4), U2.12 (PF2)
- new net POT_A: J13.4 (Pin_4)
- new net POT_B: J14.4 (Pin_4)
- new net POT_C: J15.4 (Pin_4)
- new net POT_D: J16.4 (Pin_4)
- new net PWM_A: J13.2 (Pin_2)
- new net PWM_B: J14.2 (Pin_2)
- new net PWM_C: J15.2 (Pin_2)
- new net PWM_D: J16.2 (Pin_2)
- new net SPI_MISO: TP5.1, U2.23 (PA6)
- new net SPI_SCK: TP4.1, U2.22 (PA5)
- new net SPI_SD_CS: TP7.1, U2.21 (PA4)
- new net UART2_RX: J7.1 (Pin_1), U2.56 (PD6)
- new net UART2_TX: J7.3 (Pin_3), U2.55 (PD5)
- new net USART1_RX: TP16.1, U2.61 (PB7)
- new net USART1_TX: TP14.1, U2.60 (PB6)
- new net USB_D+: J5.3 (D+), R7.2
- no-connect marks 0 -> 17
Other:
- note added: "CAN"
- note added: "Extras"
- note added: "I^{2}C"
- note added: "MCU"
- note added: "POWER INPUT"
- note added: "SERVO OUTPUTS"
- note added: "SWD"
- note added: "UART"
- note added: "USB"
- note removed: "Check that the feedback voltage is small enough for the micro"
