File: Boards/Servo_Board/Servo_Board.kicad_pcb (KiCad board)
At the start: 4 copper layers, 100 x 50 mm, 98 parts, among them J1 SWD JST PH, J10 CAN2_T, J11 I2CC JST, J12 DB9 Microfit, J14 SERVO B, J15 SERVO A, J16 SERVO C, J17 SERVO D, J18 Extras JST, J19 Backup Power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

Commit message: Completed with manufacturing files
Parts:
- added G***: LOGO, logo:uca_logo2, B.Cu at (155.6, 88.6)
- added TP16: 7.4V, TestPoint:TestPoint_Pad_D1.0mm, F.Cu at (188.6, 98.6)
- added TP17: 5V, TestPoint:TestPoint_Pad_D1.0mm, F.Cu at (176.2, 107.6)
- added TP18: 3.3V, TestPoint:TestPoint_Pad_D1.0mm, F.Cu at (157.2, 102.8)
- added TP19: GND, TestPoint:TestPoint_Bridge_Pitch2.54mm_Drill1.3mm, F.Cu at (110.1, 116.0)
- added TP20: GND, TestPoint:TestPoint_Bridge_Pitch2.54mm_Drill1.3mm, F.Cu at (155.0, 81.0)
- added TP3: 2S+, TestPoint:TestPoint_Pad_D1.0mm, F.Cu at (165.2, 95.2)
- added TP4: P_SOURCE, TestPoint:TestPoint_Pad_D1.0mm, F.Cu at (188.2, 103.0)
- TP1, TP2: footprint TestPoint:TestPoint_Pad_1.5x1.5mm -> TestPoint:TestPoint_Pad_D1.0mm
- moved TP2 84.6 mm to (142.8, 100.4)
- moved TP1 78.9 mm to (148.4, 98.4)
- moved C15 0.40 mm to (194.6, 94.8)
- moved C17 0.40 mm to (194.6, 87.4)
- moved J10 0.40 mm to (127.8, 110.2)
- moved J9 0.20 mm to (172.1, 110.2)
Routing:
- net +3V3: track 56.0 -> 70.1 mm, vias 17 -> 18
- net +5V: track 46.1 -> 55.8 mm
- net +7V4: track 133.1 -> 135.6 mm
- net /CAN1_RX: track 27.1 -> 28.9 mm
- net /PWR_SOURCE: track 71.6 -> 73.3 mm
- net /2S+ A10: track 70.4 -> 72.0 mm
- net /CAN1_TX: track 23.6 -> 25.1 mm
- net Net-(D6-K): track 22.9 -> 21.9 mm
- net GND: track 56.5 -> 57.3 mm
- net Net-(D10-A2): track 9.43 -> 10.2 mm
- net /PWM_EXT: track 17.3 -> 17.9 mm
Other:
- board text added: "${CURRENT_DATE}"
- board text added: "${REVISION}"
- board text added: "7V4"
- board text added: "B Redpath"
- board text added: "CAN IN"
- board text added: "CAN OUT"
- board text added: "Date"
- board text added: "Drawn"
- board text added: "ERR"
- board text added: "EXTRAS A"
- board text added: "EXTRAS B"
- board text added: "HYBRID SERVO ECU"
- board text added: "I^{2}C A"
- board text added: "I^{2}C B"
- board text added: "I^{2}C C"
- board text added: "PWR SWITCH"
- board text added: "REDUNDANT PWR 2S ONLY"
- board text added: "Revision"
- board text added: "SERVO A"
- board text added: "SERVO B"
- board text added: "SERVO C"
- board text added: "SERVO D"
- board text added: "SPI"
- board text added: "STATUS"
- board text added: "SWD"
- board text added: "TERM A"
- board text added: "TERM B"
- board text added: "UART"
