File: Boards/ADC_Board/ADC_Board.kicad_sch (KiCad schematic)
At the start: 87 parts, among them J1 SWD JST PH, J10 I2CC JST, J11 DB9 Microfit, J12 Backup Power, J2 UART JST, J3 Extras JST, J4 USB_B_Micro, J5 I2CA JST, J6 DB9 Microfit, J7 I2CB JST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

Commit message: Rev B ADC Board
Change ADC to QFN due to order error
Adds voltage divider to MIPA ADC lines
Parts:
- removed TP12: A9, TestPoint:TestPoint_Pad_D1.0mm, symbol Connector:TestPoint_Small
Connections:
- net A9 renamed 5VREF
Other:
- sheet Analog Domain ports: added 5VREF; removed none
Changed lines of the file:
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@@
 	(title_block
 		(title "ADC ECU Board")
-		(date "2025-05-14")
-		(rev "A")
+		(date "2025-07-15")
+		(rev "B")
 		(company "Hybrid Test Stand")
 		(comment 1 "Drawn: Brad Redpath")
@@
 	(wire
 		(pts
+			(xy 262.89 134.62) (xy 233.68 134.62)
+		)
+		(stroke
+			(width 0)
+			(type default)
+		)
+	)
+	(wire
+		(pts
+			(xy 233.68 134.62) (xy 233.68 143.51)
+		)
+		(stroke
+			(width 0)
+			(type default)
+		)
+	)
+	(wire
+		(pts
 			(xy 127 50.8) (xy 125.73 50.8)
 		)
@@
 	(wire
 		(pts
+			(xy 287.02 100.33) (xy 262.89 100.33)
+		)
+		(stroke
+			(width 0)
+			(type default)
+		)
+	)
+	(wire
+		(pts
 			(xy 326.39 157.48) (xy 354.33 157.48)
 		)
@@
 	(wire
 		(pts
-			(xy 209.55 143.51) (xy 227.33 143.51)
+			(xy 209.55 143.51) (xy 233.68 143.51)
 		)
 		(stroke
@@
 	(wire
 		(pts
+			(xy 262.89 100.33) (xy 262.89 134.62)
+		)
+		(stroke
+			(width 0)
+			(type default)
+		)
+	)
+	(wire
+		(pts
 			(xy 140.97 118.11) (xy 153.67 118.11)
 		)
@@
 		)
 	)
-	(label "A9"
-		(at 222.25 143.51 180)
-		(effects
-			(font
-				(size 1.27 1.27)
-			)
-			(justify right bottom)
-		)
-	)
 	(label "LED1"
 		(at 106.68 250.19 180)
@@
 		)
 	)
+	(label "5VREF"
+		(at 222.25 143.51 180)
+		(effects
+			(font
+				(size 1.27 1.27)
+			)
+			(justify right bottom)
+		)
+	)
 	(label "MIPA_B A2"
 		(at 222.25 102.87 180)
@@
 	)
 	(symbol
-		(lib_id "Connector:TestPoint_Small")
-		(at 227.33 143.51 270)
-		(mirror x)
-		(unit 1)
-		(exclude_from_sim no)
-		(in_bom yes)
-		(on_board yes)
-		(dnp no)
-		(fields_autoplaced yes)
-		(property "Reference" "TP12"
-			(at 228.6 142.2399 90)
-			(effects
-				(font
-					(size 1.27 1.27)
-				)
-				(justify left)
-			)
-		)
-		(property "Value" "A9"
-			(at 228.6 144.7799 90)
-			(effects
-				(font
-					(size 1.27 1.27)
-				)
-				(justify left)
-			)
-		)
-		(property "Footprint" "TestPoint:TestPoint_Pad_D1.0mm"
-			(at 227.33 138.43 0)
-			(effects
-				(font
-					(size 1.27 1.27)
-				)
-				(hide yes)
-			)
-		)
-		(property "Datasheet" "~"
-			(at 227.33 138.43 0)
-			(effects
-				(font
-					(size 1.27 1.27)
-				)
-				(hide yes)
-			)
-		)
-		(property "Description" "test point"
-			(at 227.33 143.51 0)
-			(effects
-				(font
-					(size 1.27 1.27)
-				)
-				(hide yes)
-			)
-		)
-		(property "Sim.Type" ""
-			(at 227.33 143.51 0)
-			(effects
-				(font
-					(size 1.27 1.27)
-				)
-			)
-		)
-		(property "Part Number" ""
-			(at 227.33 143.51 0)
-			(effects
-				(font
-					(size 1.27 1.27)
-				)
-			)
-		)
-		(pin "1"
-		)
-		(instances
-			(project "ADC_Board"
-				(path "/4595bb47-7b8a-406e-962e-ec9ceed32faf"
-					(reference "TP12")
-					(unit 1)
-				)
-			)
-		)
-	)
-	(symbol
 		(lib_id "power:+3V3")
 		(at 25.4 95.25 0)
@@
 			(effects
 				(font
+					(size 1.27 1.27)
+				)
+				(justify left)
+			)
+		)
+		(pin "5VREF" output
+			(at 287.02 100.33 180)
+			(effects
+				(font
